File: Projects/[2]AI7688H.sch (KiCad schematic (older format))
At the start: 103 parts, among them CON1 TF-Micro-SDCard, J1 CONN_SMA, P1 USB_OTG, P10 CONN_01X04, P2 USB_A, P3 HR911102A, P4 CONN_01X14, P5 CONN_01X12, P6 CONN_01X04, P7 CONN_01X16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

Commit message: fix footprint cp2102
Parts:
- U1: footprint nhantt-kicad-lib:QFN-32-1EP_5x5mm_Pitch0.5mm -> Housings_DFN_QFN:QFN-28-1EP_5x5mm_Pitch0.5mm
Changed lines of the file:
@@
 F 0 "U1" H 4375 8015 50  0000 C CNN
 F 1 "CP2102" H 4375 7924 50  0000 C CNN
-F 2 "nhantt-kicad-lib:QFN-32-1EP_5x5mm_Pitch0.5mm" H 4325 7350 60  0001 C CNN
+F 2 "Housings_DFN_QFN:QFN-28-1EP_5x5mm_Pitch0.5mm" H 4325 7350 60  0001 C CNN
 F 3 "" H 4325 7350 60  0001 C CNN
 	1    4325 7350
